Commit message: added gelsight_vision meshes and config (non-calibrated)

File: rgt_manager/urdf/rgt.urdf (robot description, URDF)
Before this commit: robot rgt, 9 links, 8 joints
Links:
- added link gelsight_vision; visual mesh filename=package://rgt_manager/meshes/gelsight_vision.glb scale=1 1 1
- added link nex10_tray_3; visual mesh filename=package://rgt_manager/meshes/tray.glb scale=1 1 1
- added link ur20_tray_3; visual mesh filename=package://rgt_manager/meshes/tray.glb scale=1 1 1
Joints:
- added joint gelsight_vision: type fixed, parent world, child gelsight_vision
- added joint nex10_tray_3: type fixed, parent world, child nex10_tray_3
- added joint ur20_tray_3: type fixed, parent world, child ur20_tray_3

Commit message: added table to urdf and rgt_manager

File: rgt_manager/urdf/rgt.urdf (robot description, URDF)
Before this commit: robot rgt, 12 links, 11 joints
Links:
- added link table; visual mesh filename=package://rgt_manager/meshes/table.glb scale=1 1 1
Joints:
- added joint table: type fixed, parent world, child table
