Commit message: added gripper connector mesh and config

File: rgt_manager/urdf/gripper.macro.xacro (robot description, xacro)
@@ -2,232 +2,15 @@
 <robot xmlns:xacro="http://ros.org/wiki/xacro">
   <xacro:macro name="gripper" params="name:=gripper parent:=world">
-    <!-- fingers links macros -->
-    <xacro:macro name="outer_knuckle" params="fingerprefix">
-      <link name="${fingerprefix}_outer_knuckle">
-        <inertial>
-          <origin xyz="-0.000200000000003065 0.0199435877845359 0.0292245259211331" rpy="0 0 0" />
-          <mass value="0.013" />
-          <inertia ixx="2.89328108496468E-06" ixy="-1.57935047237397E-19" ixz="-1.93980378593255E-19" iyy="1.86719750325683E-06" iyz="-1.21858577871576E-06" izz="1.21905238907251E-06" />
-        </inertial>
-        <visual>
-          <origin xyz="0 0 0" rpy="0 0 0" />
-          <geometry>
-            <mesh filename="package://rgt_manager/meshes/gripper/visual/outer_knuckle.stl" />
-          </geometry>
-          <material name="">
-            <color rgba="0.65 0.65 0.65 1" />
-          </material>
-        </visual>
-        <collision>
-          <origin xyz="0 0 0" rpy="0 0 0" />
-          <geometry>
-            <mesh filename="package://rgt_manager/meshes/gripper/collision/outer_knuckle.stl"/>
-          </geometry>
-        </collision>
-      </link>
-    </xacro:macro>
-    <xacro:macro name="bar" params="fingerprefix">
-      <link name="${fingerprefix}_bar">
-        <inertial>
-          <origin xyz="0.00030115855001899 0.0373907951953854 -0.0208027427000385" rpy="0 0 0" />
-          <mass value="0.041" />
-          <inertia ixx="1.52518312458174E-05" ixy="9.76583423954399E-10" ixz="-5.43838577022588E-10" iyy="6.17694243867776E-06" iyz="6.78636130740228E-06" izz="1.16494917907219E-05" />
-        </inertial>
-        <visual>
-          <origin xyz="0 0 0" rpy="0 0 0" />
-          <geometry>
-            <mesh filename="package://rgt_manager/meshes/gripper/visual/bar.stl" />
-          </geometry>
-          <material name="">
-            <color rgba="0.13 0.13 0.13 1" />
-          </material>
-        </visual>
-        <collision>
-          <origin xyz="0 0 0" rpy="0 0 0" />
-          <geometry>
-            <mesh filename="package://rgt_manager/meshes/gripper/collision/bar.stl" />
-          </geometry>
-        </collision>
-      </link>
-    </xacro:macro>
-    <xacro:macro name="proximal_phalanx" params="fingerprefix">
-      <link name="${fingerprefix}_proximal_phalanx">
-        <inertial>
-          <origin xyz="0.000123011831763771 0.0507850843201817 0.00103968640075166" rpy="0 0 0" />
-          <mass value="0.028" />
-          <inertia ixx="2.61910379223783E-05" ixy="-2.43616858946494E-07" ixz="-6.37789906117123E-09" iyy="2.8270243746167E-06" iyz="-5.37200748039765E-07" izz="2.83695868220296E-05" />
-        </inertial>
-        <visual>
-          <origin xyz="0 0 0" rpy="0 0 0" />
-          <geometry>
-            <mesh filename="package://rgt_manager/meshes/gripper/visual/proximal_phalanx.stl" />
-          </geometry>
-          <material name="">
-            <color rgba="0.13 0.13 0.13 1" />
-          </material>
-        </visual>
-        <collision>
-          <origin xyz="0 0 0" rpy="0 0 0" />
-          <geometry>
-            <mesh filename="package://rgt_manager/meshes/gripper/collision/proximal_phalanx.stl" />
-          </geometry>
-        </collision>
-      </link>
-    </xacro:macro>
-    <xacro:macro name="distal_phalanx" params="fingerprefix">
-      <link name="${fingerprefix}_distal_phalanx">
-        <inertial>
-          <origin xyz="0 -0.009 0.005" rpy="0 0 0" />
-          <mass value="0.02" />
-          <inertia ixx="1.839e-6" ixy="2.943e-15" ixz="-8.887e-15" iyy="1.184e-6" iyz="4.328e-7" izz="1.820e-6" />
-        </inertial>
-        <visual>
-          <origin xyz="0 0 0" rpy="0 0 0" />
-          <geometry>
-            <mesh filename="package://rgt_manager/meshes/gripper/visual/driver.dae" />
-          </geometry>
-          <material name="">
-            <color rgba="0.13 0.13 0.13 1" />
-          </material>
-        </visual>
-        <collision>
-          <origin xyz="0 0 0" rpy="0 0 0" />
-          <geometry>
-            <mesh filename="package://rgt_manager/meshes/gripper/collision/driver.stl" />
-          </geometry>
-        </collision>
-      </link>
-    </xacro:macro>
-    <xacro:macro name="finger_tip" params="fingerprefix">
-      <link name="${fingerprefix}_finger_tip">
-        <inertial>
-          <origin xyz="0 -0.008 0.016" rpy="0 0 0" />
-          <mass value="0.021" />
-          <inertia ixx="3.071e-6" ixy="-3.735e-13" ixz="-1.785e-13" iyy="3.467e-6" iyz="4.052e-7" izz="1.175e-6" />
-        </inertial>
-        <visual>
-          <origin xyz="0 0 0" rpy="0 0 0" />
-          <geometry>
-            <mesh filename="package://rgt_manager/meshes/gripper/visual/agc-tip-mld-kit-85.dae" />
-          </geometry>
-        </visual>
-        <collision>
-          <origin xyz="0 0 0" rpy="0 0 0" />
-          <geometry>
-            <mesh filename="package://rgt_manager/meshes/gripper/collision/agc-tip-mld-kit-85.stl" />
-          </geometry>
-        </collision>
-      </link>
-    </xacro:macro>
-    <xacro:macro name="finger_links" params="fingerprefix">
-      <xacro:outer_knuckle fingerprefix="${fingerprefix}"/>
-      <xacro:bar fingerprefix="${fingerprefix}"/>
-      <xacro:distal_phalanx fingerprefix="${fingerprefix}"/>
-      <xacro:finger_tip fingerprefix="${fingerprefix}"/>
-      <xacro:proximal_phalanx fingerprefix="${fingerprefix}"/>
-    </xacro:macro>
-    <!-- fingers joints macros -->
-    <xacro:macro name="bar_joint" params="fingerprefix">
-      <joint name="${fingerprefix}_bar_joint" type="fixed">
-        <origin xyz="0 0.0315 -0.0041" rpy="0 0 0"/>
-        <parent link="${fingerprefix}_outer_knuckle" />
-        <child link="${fingerprefix}_bar" />
-        <axis xyz="1 0 0" />
-      </joint>
-    </xacro:macro>
-    <xacro:macro name="proximal_phalanx_joint" params="fingerprefix reflect">
-      <joint name="${fingerprefix}_proximal_phalanx_joint" type="revolute">
-        <origin xyz="0 ${reflect * -0.0127} 0.06142" rpy=".125 0 ${(1 + reflect) * pi / 2}"/>
-        <parent link="robotiq_arg2f_base_link" />
-        <child link="${fingerprefix}_proximal_phalanx" />
-        <axis xyz="1 0 0" />
-        <limit lower="0" upper="0.8757" velocity="0.5" effort="1000" />
-        <mimic joint="finger_joint" multiplier="1" offset="0" />
-      </joint>
-    </xacro:macro>
-    <xacro:macro name="distal_phalanx_joint" params="fingerprefix">
-      <joint name="${fingerprefix}_distal_phalanx_joint" type="revolute">
-        <origin xyz="0 0.0061 0.0471" rpy="0 0 0"/>
-        <parent link="${fingerprefix}_bar" />
-        <child link="${fingerprefix}_distal_phalanx" />
-        <axis xyz="1 0 0" />
-        <limit lower="-0.8757" upper="0" velocity="0.5" effort="1000" />
-        <mimic joint="finger_joint" multiplier="-1" offset="0" />
-      </joint>
-    </xacro:macro>
-    <xacro:macro name="finger_tip_joint" params="fingerprefix">
-      <joint name="${fingerprefix}_finger_tip_joint" type="fixed">
-        <origin xyz="0 -0.011402 0.01305" rpy="0 0 0"/>
-        <parent link="${fingerprefix}_distal_phalanx" />
-        <child link="${fingerprefix}_finger_tip" />
-      </joint>
-    </xacro:macro>
-    <xacro:macro name="finger_joints" params="fingerprefix reflect">
-      <xacro:bar_joint fingerprefix="${fingerprefix}"/>
-      <xacro:proximal_phalanx_joint fingerprefix="${fingerprefix}" reflect="${reflect}"/>
-      <xacro:distal_phalanx_joint fingerprefix="${fingerprefix}"/>
-      <xacro:finger_tip_joint fingerprefix="${fingerprefix}"/>
-      <!-- <xacro:pad_joint fingerprefix="${fingerprefix}"/> -->
-    </xacro:macro>
-    <!-- base link -->
-    <link name="${name}" />
-    <joint name="${name}_to_robotiq_arg2f_base_link" type="fixed">
-      <parent link="${name}" />
-      <child link="robotiq_arg2f_base_link" />
-    </joint>
+    <link name="${name}">
+      <visual>
+        <geometry>
+          <mesh filename="package://rgt_manager/meshes/gripper_connector.glb" scale="1 1 1" />
+        </geometry>
+      </visual>
+    </link>
     <joint name="${name}" type="fixed">
       <parent link="${parent}" />
       <child link="${name}" />
     </joint>
-    <link name="robotiq_arg2f_base_link">
-        <inertial>
-          <origin xyz="8.625E-08 -4.6583E-06 0.03145" rpy="0 0 0" />
-          <mass value="0.635" />
-          <inertia ixx="0.000494023" ixy="0.0" ixz="0.0" iyy="0.000562779" iyz="0.0" izz="0.000377692" />
-        </inertial>
-        <visual>
-          <origin xyz="0 0 0" rpy="0 0 0" />
-          <geometry>
-            <mesh filename="package://rgt_manager/meshes/gripper/visual/base_link.dae" />
-          </geometry>
-          <material name="">
-            <color rgba="0.13 0.13 0.13 1" />
-          </material>
-        </visual>
-        <collision>
-          <origin xyz="0 0 0" rpy="0 0 0" />
-          <geometry>
-            <mesh filename="package://rgt_manager/meshes/gripper/collision/base_link.stl" />
-          </geometry>
-        </collision>
-      </link>
-    <!-- TCP frame centered between the fingers near the grasp equilibrium point -->
-    <link name="robotiq_arg2f_tcp"/>
-    <joint name="robotiq_arg2f_tcp_joint" type="fixed">
-      <origin rpy="0 0 0" xyz="0 0 0.174"/>
-      <parent link="robotiq_arg2f_base_link"/>
-      <child link="robotiq_arg2f_tcp"/>
-    </joint>
-    <!-- left finger -->
-    <xacro:finger_links fingerprefix="left"/>
-    <xacro:finger_joints fingerprefix="left" reflect="1.0"/>
-    <joint name="finger_joint" type="revolute">
-      <origin xyz="0 -0.0306011 0.054904" rpy="0 0 ${pi}"/>
-      <parent link="robotiq_arg2f_base_link" />
-      <child link="left_outer_knuckle" />
-      <axis xyz="1 0 0" />
-      <limit lower="0" upper="0.8" velocity="0.5" effort="1000" />
-    </joint>
-    <!-- right finger -->
-    <xacro:finger_joints fingerprefix="right" reflect="-1.0"/>
-    <xacro:finger_links fingerprefix="right"/>
-    <joint name="right_finger_joint" type="revolute">
-      <origin xyz="0 0.0306011 0.054904" rpy="0 0 0"/>
-      <parent link="robotiq_arg2f_base_link" />
-      <child link="right_outer_knuckle" />
-      <axis xyz="1 0 0" />
-      <limit lower="0" upper="0.81" velocity="0.5" effort="1000" />
-      <mimic joint="finger_joint" multiplier="1" offset="0" />
-    </joint>
   </xacro:macro>
 </robot>

File: rgt_manager/urdf/rgt.xacro (robot description, xacro)
@@ -8,5 +8,5 @@
   <xacro:include filename="$(find rgt_manager)/urdf/grinder.macro.xacro" />
   <xacro:include filename="$(find rgt_manager)/urdf/gelsight_vision.macro.xacro" />
-  <!-- <xacro:include filename="$(find rgt_manager)/urdf/gripper.macro.xacro" /> -->
+  <xacro:include filename="$(find rgt_manager)/urdf/gripper.macro.xacro" />
   <xacro:include filename="$(find rgt_manager)/urdf/table.macro.xacro" />
   <!-- Base Link -->
@@ -19,12 +19,14 @@
   <xacro:tray name="nex10_tray_2" />
   <xacro:tray name="nex10_tray_3" />
+  <xacro:tray name="nex10_tray_4" />
   <xacro:tray name="ur20_tray_1" />
   <xacro:tray name="ur20_tray_2" />
   <xacro:tray name="ur20_tray_3" />
+  <xacro:tray name="ur20_tray_4" />
   <!-- Tools -->
   <xacro:sander />
   <xacro:grinder />
   <xacro:gelsight_vision />
-  <!-- <xacro:gripper /> -->
+  <xacro:gripper />
   <!-- Table -->
   <xacro:table />
